Commit message: added meshes

File: robots/fr3.urdf (robot description, URDF)
Before this commit: robot fr3, 17 links, 16 joints
Links:
- link fr3_link0: geometry collision mesh filename=meshes/collision/link0.stl; visual mesh filename=meshes/visual/link0.dae
- link fr3_link1: geometry collision mesh filename=meshes/collision/link1.stl; visual mesh filename=meshes/visual/link1.dae
- link fr3_link2: geometry collision mesh filename=meshes/collision/link2.stl; visual mesh filename=meshes/visual/link2.dae
- link fr3_link3: geometry collision mesh filename=meshes/collision/link3.stl; visual mesh filename=meshes/visual/link3.dae
- link fr3_link4: geometry collision mesh filename=meshes/collision/link4.stl; visual mesh filename=meshes/visual/link4.dae
- link fr3_link5: geometry collision mesh filename=meshes/collision/link5.stl; visual mesh filename=meshes/visual/link5.dae
- link fr3_link6: geometry collision mesh filename=meshes/collision/link6.stl; visual mesh filename=meshes/visual/link6.dae
- link fr3_link7: geometry collision mesh filename=meshes/collision/link7.stl; visual mesh filename=meshes/visual/link7.dae

Commit message: updated urdf file

File: robots/fr3.urdf (robot description, URDF)
Before this commit: robot fr3, 17 links, 16 joints
Links:
- removed link fr3_link0_sc
- removed link fr3_link1_sc
- removed link fr3_link2_sc
- removed link fr3_link3_sc
- removed link fr3_link4_sc
- removed link fr3_link5_sc
- removed link fr3_link6_sc
- removed link fr3_link7_sc
- added link fr3_hand, mass 0.73; collision mesh filename=meshes/collision/hand.stl; visual mesh filename=meshes/visual/hand.dae
- added link fr3_hand_tcp, mass 0.0
- added link fr3_leftfinger, mass 0.015; collision box size=17.5e-3 15.2e-3 18.5e-3; collision box size=17.5e-3 7e-3 23.5e-3
- added link fr3_rightfinger, mass 0.015; collision box size=17.5e-3 15.2e-3 18.5e-3; collision box size=17.5e-3 7e-3 23.5e-3
- added link world
- link fr3_link0: mass None -> 0.629769
- link fr3_link1: mass None -> 4.970684
- link fr3_link2: mass None -> 0.646926
- link fr3_link3: mass None -> 3.228604
- link fr3_link4: mass None -> 3.587895
- link fr3_link5: mass None -> 1.225946
- link fr3_link6: mass None -> 1.666555
- link fr3_link7: mass None -> 0.735522
- link fr3_link8: mass None -> 0.0
Joints:
- removed joint fr3_link0_sc_joint
- removed joint fr3_link1_sc_joint
- removed joint fr3_link2_sc_joint
- removed joint fr3_link3_sc_joint
- removed joint fr3_link4_sc_joint
- removed joint fr3_link5_sc_joint
- removed joint fr3_link6_sc_joint
- removed joint fr3_link7_sc_joint
- added joint fr3_finger_joint1: type prismatic, parent fr3_hand, child fr3_leftfinger, origin xyz=0 0 0.0584 rpy=0 0 0, axis 0 1 0, limit lower=0.0 upper=0.04 effort=100 velocity=0.2
- added joint fr3_finger_joint2: type prismatic, parent fr3_hand, child fr3_rightfinger, origin xyz=0 0 0.0584 rpy=0 0 0, axis 0 -1 0, limit lower=0.0 upper=0.04 effort=100 velocity=0.2, mimic joint=fr3_finger_joint1
- added joint fr3_hand_joint: type fixed, parent fr3_link8, child fr3_hand, origin xyz=0 0 0 rpy=0 0 -0.7853981633974483
- added joint fr3_hand_tcp_joint: type fixed, parent fr3_hand, child fr3_hand_tcp, origin xyz=0 0 0.1034 rpy=0 0 0
- added joint world_joint: type fixed, parent world, child fr3_link0, origin xyz=0 0 0 rpy=0 0 0

Commit message: updated urdf file

File: robots/fr3.urdf (robot description, URDF)
Before this commit: robot fr3, 14 links, 13 joints
Links:
- removed link world
- link fr3_hand: geometry collision mesh filename=./meshes/collision/hand.stl; visual mesh filename=./meshes/visual/hand.obj
- link fr3_hand_tcp: mass 0.0 -> None
- link fr3_leftfinger: geometry collision box size=17.5e-3 15.2e-3 18.5e-3; collision box size=17.5e-3 7e-3 23.5e-3
- link fr3_link0: geometry collision mesh filename=./meshes/collision/link0.stl; visual mesh filename=./meshes/visual/link0.obj
- link fr3_link1: geometry collision mesh filename=./meshes/collision/link1.stl; visual mesh filename=./meshes/visual/link1.obj
- link fr3_link2: geometry collision mesh filename=./meshes/collision/link2.stl; visual mesh filename=./meshes/visual/link2.obj
- link fr3_link3: geometry collision mesh filename=./meshes/collision/link3.stl; visual mesh filename=./meshes/visual/link3.obj
- link fr3_link4: geometry collision mesh filename=./meshes/collision/link4.stl; visual mesh filename=./meshes/visual/link4.obj
- link fr3_link5: geometry collision mesh filename=./meshes/collision/link5.stl; visual mesh filename=./meshes/visual/link5.obj
- link fr3_link6: geometry collision mesh filename=./meshes/collision/link6.stl; visual mesh filename=./meshes/visual/link6.obj
- link fr3_link7: geometry collision mesh filename=./meshes/collision/link7.stl; visual mesh filename=./meshes/visual/link7.obj
- link fr3_link8: mass 0.0 -> None
- link fr3_rightfinger: geometry collision box size=17.5e-3 15.2e-3 18.5e-3; collision box size=17.5e-3 7e-3 23.5e-3
Joints:
- removed joint world_joint

Commit message: updated urdf to be compatible with pinocchio (no link with unspecified mass and inertia)

File: robots/fr3.urdf (robot description, URDF)
Before this commit: robot fr3, 13 links, 12 joints
Links:
- link fr3_hand_tcp: mass None -> 0.0
- link fr3_link8: mass None -> 0.0
