Commit message: enabled installation

File: FR3Env/robots/fr3.urdf (robot description, URDF)
Before this commit: robot fr3, 13 links, 12 joints
Links:
- link fr3_hand: geometry collision mesh filename=/Users/bolundai/miniconda3/envs/mim_env/lib/python3.8/site-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; visual mesh filename=/Users/bolundai/miniconda3/envs/mim_env/lib/python3.8/site-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
- link fr3_leftfinger: geometry collision box size=17.5e-3 15.2e-3 18.5e-3; collision box size=17.5e-3 7e-3 23.5e-3
- link fr3_link0: geometry collision mesh filename=/Users/bolundai/miniconda3/envs/mim_env/lib/python3.8/site-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; visual mesh filename=/Users/bolundai/miniconda3/envs/mim_env/lib/python3.8/site-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
- link fr3_link1: geometry collision mesh filename=/Users/bolundai/miniconda3/envs/mim_env/lib/python3.8/site-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; visual mesh filename=/Users/bolundai/miniconda3/envs/mim_env/lib/python3.8/site-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
- link fr3_link2: geometry collision mesh filename=/Users/bolundai/miniconda3/envs/mim_env/lib/python3.8/site-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; visual mesh filename=/Users/bolundai/miniconda3/envs/mim_env/lib/python3.8/site-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
- link fr3_link3: geometry collision mesh filename=/Users/bolundai/miniconda3/envs/mim_env/lib/python3.8/site-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; visual mesh filename=/Users/bolundai/miniconda3/envs/mim_env/lib/python3.8/site-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
- link fr3_link4: geometry collision mesh filename=/Users/bolundai/miniconda3/envs/mim_env/lib/python3.8/site-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; visual mesh filename=/Users/bolundai/miniconda3/envs/mim_env/lib/python3.8/site-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
- link fr3_link5: geometry collision mesh filename=/Users/bolundai/miniconda3/envs/mim_env/lib/python3.8/site-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; visual mesh filename=/Users/bolundai/miniconda3/envs/mim_env/lib/python3.8/site-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
- link fr3_link6: geometry collision mesh filename=/Users/bolundai/miniconda3/envs/mim_env/lib/python3.8/site-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; visual mesh filename=/Users/bolundai/miniconda3/envs/mim_env/lib/python3.8/site-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
- link fr3_link7: geometry collision mesh filename=/Users/bolundai/miniconda3/envs/mim_env/lib/python3.8/site-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; visual mesh filename=/Users/bolundai/miniconda3/envs/mim_env/lib/python3.8/site-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
- link fr3_rightfinger: geometry collision box size=17.5e-3 15.2e-3 18.5e-3; collision box size=17.5e-3 7e-3 23.5e-3

Commit message: local changes

File: FR3Env/robots/fr3.urdf (robot description, URDF)
Before this commit: robot fr3, 13 links, 12 joints
Links:
- link fr3_hand: geometry collision mesh filename=/home/bolun/Documents/FR3Env/FR3Env/robots/meshes/collision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; visual mesh filename=/home/bolun/Documents/FR3Env/FR3Env/robots/meshes/visual/ha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
- link fr3_leftfinger: geometry collision box size=17.5e-3 15.2e-3 18.5e-3; collision box size=17.5e-3 7e-3 23.5e-3
- link fr3_link0: geometry collision mesh filename=/home/bolun/Documents/FR3Env/FR3Env/robots/meshes/collision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; visual mesh filename=/home/bolun/Documents/FR3Env/FR3Env/robots/meshes/visual/li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
- link fr3_link1: geometry collision mesh filename=/home/bolun/Documents/FR3Env/FR3Env/robots/meshes/collision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; visual mesh filename=/home/bolun/Documents/FR3Env/FR3Env/robots/meshes/visual/li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
- link fr3_link2: geometry collision mesh filename=/home/bolun/Documents/FR3Env/FR3Env/robots/meshes/collision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; visual mesh filename=/home/bolun/Documents/FR3Env/FR3Env/robots/meshes/visual/li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
- link fr3_link3: geometry collision mesh filename=/home/bolun/Documents/FR3Env/FR3Env/robots/meshes/collision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; visual mesh filename=/home/bolun/Documents/FR3Env/FR3Env/robots/meshes/visual/li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
- link fr3_link4: geometry collision mesh filename=/home/bolun/Documents/FR3Env/FR3Env/robots/meshes/collision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; visual mesh filename=/home/bolun/Documents/FR3Env/FR3Env/robots/meshes/visual/li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
- link fr3_link5: geometry collision mesh filename=/home/bolun/Documents/FR3Env/FR3Env/robots/meshes/collision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; visual mesh filename=/home/bolun/Documents/FR3Env/FR3Env/robots/meshes/visual/li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
- link fr3_link6: geometry collision mesh filename=/home/bolun/Documents/FR3Env/FR3Env/robots/meshes/collision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; visual mesh filename=/home/bolun/Documents/FR3Env/FR3Env/robots/meshes/visual/li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
- link fr3_link7: geometry collision mesh filename=/home/bolun/Documents/FR3Env/FR3Env/robots/meshes/collision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; visual mesh filename=/home/bolun/Documents/FR3Env/FR3Env/robots/meshes/visual/li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
- link fr3_rightfinger: geometry collision box size=17.5e-3 15.2e-3 18.5e-3; collision box size=17.5e-3 7e-3 23.5e-3

Commit message: pinocchio added mesh path

File: FR3Env/robots/fr3.urdf (robot description, URDF)
Before this commit: robot fr3, 13 links, 12 joints
Links:
- link fr3_hand: geometry collision mesh filename=package://robots/meshes/collision/hand.stl; visual mesh filename=package://robots/meshes/visual/hand.obj
- link fr3_leftfinger: geometry collision box size=17.5e-3 15.2e-3 18.5e-3; collision box size=17.5e-3 7e-3 23.5e-3
- link fr3_link0: geometry collision mesh filename=package://robots/meshes/collision/link0.stl; visual mesh filename=package://robots/meshes/visual/link0.obj
- link fr3_link1: geometry collision mesh filename=package://robots/meshes/collision/link1.stl; visual mesh filename=package://robots/meshes/visual/link1.obj
- link fr3_link2: geometry collision mesh filename=package://robots/meshes/collision/link2.stl; visual mesh filename=package://robots/meshes/visual/link2.obj
- link fr3_link3: geometry collision mesh filename=package://robots/meshes/collision/link3.stl; visual mesh filename=package://robots/meshes/visual/link3.obj
- link fr3_link4: geometry collision mesh filename=package://robots/meshes/collision/link4.stl; visual mesh filename=package://robots/meshes/visual/link4.obj
- link fr3_link5: geometry collision mesh filename=package://robots/meshes/collision/link5.stl; visual mesh filename=package://robots/meshes/visual/link5.obj
- link fr3_link6: geometry collision mesh filename=package://robots/meshes/collision/link6.stl; visual mesh filename=package://robots/meshes/visual/link6.obj
- link fr3_link7: geometry collision mesh filename=package://robots/meshes/collision/link7.stl; visual mesh filename=package://robots/meshes/visual/link7.obj
- link fr3_rightfinger: geometry collision box size=17.5e-3 15.2e-3 18.5e-3; collision box size=17.5e-3 7e-3 23.5e-3
