Commit message: added loading of crude model

File: FR3Env/robots/fr3_crude.urdf (robot description, URDF)
Before this commit: robot fr3, 13 links, 12 joints
Links:
- link fr3_leftfinger: geometry collision box size=17.5e-3 15.2e-3 18.5e-3; collision box size=17.5e-3 7e-3 23.5e-3
- link fr3_link8: mass None -> 1e-5
- link fr3_rightfinger: geometry collision box size=17.5e-3 15.2e-3 18.5e-3; collision box size=17.5e-3 7e-3 23.5e-3

Commit message: updated crude urdf

File: FR3Env/robots/fr3_crude.urdf (robot description, URDF)
Before this commit: robot fr3, 13 links, 12 joints
Links:
- link fr3_hand: geometry collision box size=0.14 0.24 0.18; visual box size=0.16 0.24 0.18
- link fr3_hand_tcp: mass None -> 1e-5
- link fr3_leftfinger: geometry 
- link fr3_link5: geometry collision cylinder length=0.25 radius=0.055; collision cylinder length=0.28 radius=0.09
- link fr3_link6: geometry collision cylinder length=0.20 radius=0.08; visual cylinder length=0.20 radius=0.08
- link fr3_link7: geometry collision cylinder length=0.28 radius=0.07; visual cylinder length=0.28 radius=0.07
- link fr3_rightfinger: geometry 
