Commit message: commented bounding box visuals

File: FR3Env/robots/fr3_with_bounding_boxes.urdf (robot description, URDF)
Before this commit: robot fr3, 20 links, 19 joints
Links:
- link fr3_hand_bounding_box: geometry 
- link fr3_link3_bounding_box: geometry 
- link fr3_link4_bounding_box: geometry 
- link fr3_link5_1_bounding_box: geometry 
- link fr3_link5_2_bounding_box: geometry 
- link fr3_link6_bounding_box: geometry 
- link fr3_link7_bounding_box: geometry 

Commit message: updated fr3_with_bounding_boxes.urdf

File: FR3Env/robots/fr3_with_bounding_boxes.urdf (robot description, URDF)
Before this commit: robot fr3, 20 links, 19 joints
Joints:
- joint fr3_hand_bounding_box_joint: origin xyz=0 0.00 0.06 rpy=0 0 0 -> xyz=0 0.00 0.04 rpy=0 0 0
